File: SIM800C.sch (KiCad schematic (older format))
At the start: 71 parts, among them J1 SIM_Card, J2 1x8, J3 SJ-2504A-SMT-TR, J4 USB_OTG, J5 U.FL-R-SMT(10), J6 Conn_01x07_Male, Q1 BJT, Q2 BJT, Q3 BJT, Q4 BJT, Q5 BJT, SW1 POWER, U1 SIM800C, U2 LM2576

Commit message: Gold fingers added
Parts:
- removed C10, C11, C12, C13, C14: 33pF, Capacitors_SMD:C_0402, symbol C_Small
- removed C19, C20: DNP, Capacitors_SMD:C_0402, symbol C_Small
- removed C9: 10pF, Capacitors_SMD:C_0402, symbol C_Small
- removed J2: 1x8, Pin_Headers:Pin_Header_Straight_1x08_Pitch2.54mm, symbol Conn_01x08
- removed J3: SJ-2504A-SMT-TR, CUI_SJ-2504A-SMT-TR, symbol SJ-2504A-SMT-TR
- removed J4: USB_OTG, symbol USB_OTG
- removed J6: Conn_01x07_Male, symbol Conn_01x07_Male
- removed Q4, Q5: BJT, symbol 2N3055
- removed R10, R7, R9: 1K, Resistors_SMD:R_0402, symbol R_Small
- removed R12: 68R, Resistors_SMD:R_0402, symbol R_Small
- removed R13: 5.6K, Resistors_SMD:R_0402, symbol R_Small
- removed R25, R26, R28, R31: 4.7K, Resistors_SMD:R_0402, symbol R_Small
- removed R27: 0R, Resistors_SMD:R_0402, symbol R_Small
- removed R29, R30: 47K, Resistors_SMD:R_0402, symbol R_Small
- added D5: ESDA6V1-5W6, TO_SOT_Packages_SMD:SOT-23-6, symbol ESDA6V1-5W6
- added J2: RPi, Pin_Headers:Pin_Header_Straight_2x07_Pitch2.54mm, symbol Conn_02x07_Odd_Even
- added J7: Conn_01x02, Pin_Headers:Pin_Header_Angled_1x02_Pitch2.54mm, symbol Conn_01x02
- added SW2: SW_SPDT, footprints:Switch-SW_SPDT_PCM12, symbol SW_SPDT
- added U3: MPCIE-Socket, footprints:mpcie-full-card, symbol MPCIE-Socket
- C1: footprint Capacitors_SMD:C_0402 -> Capacitors_Tantalum_SMD:CP_Tantalum_Case-C_EIA-6032-28_Reflow
- C17: renamed from C15; footprint Capacitors_SMD:C_0402 -> Capacitors_SMD:CP_Elec_6.3x7.7
- C18: renamed from C16; footprint Capacitors_SMD:C_0402 -> Capacitors_SMD:C_0603
- C19: renamed from C17; footprint Capacitors_SMD:C_0402 -> Capacitors_SMD:CP_Elec_6.3x7.7
- C2: footprint Capacitors_SMD:C_0402 -> Capacitors_SMD:C_0603
- C7, C8: value 10pF -> DNP
- D1: footprint (none) -> Diodes_SMD:D_SOD-123
- D2, D3: footprint (none) -> LEDs:LED_0402
- D4: footprint (none) -> Diodes_SMD:D_SMA
- J1: footprint (none) -> footprints:L-KLS1-SIM-064-(6+2)P-H1
- J6: renamed from J5; footprint HRS_U.FL-R-SMT(10) -> U.FL-R-SMT_10_:HRS_U.FL-R-SMT(10)
- L1: footprint (none) -> Inductors_SMD:L_6.3x6.3_H3
- L2: footprint (none) -> Inductors_SMD:L_0805
- Q1, Q2, Q3: footprint (none) -> TO_SOT_Packages_SMD:SOT-23
- R16: value 47K -> 4.7K
- R18: value 1K -> 4.7K
- R19: value 1K -> 47K
- R23: renamed from R22; value 1K -> 4.7K
- R24: renamed from R23; value 1K -> 47K
- R6: value 1K -> 0R
- SW1: footprint (none) -> footprints:Buton-SW_SPST_B3U-1000P
- U1: footprint LCC110P1570X1760X250-42N -> SIM800C:LCC110P1570X1760X250-42N
- U2: footprint (none) -> TO_SOT_Packages_SMD:TO-263-5_TabPin3
- renumbered C18 to C20, R20 to R21, R21 to R22, R24 to R25
Connections:
- net GND: now also C7.2, C8.2, J6.GND1 (GND), J6.GND2 (GND), D5.1, D5.2, D5.3, J2.14 (Pin_14), J2.6 (Pin_6), J2.9 (Pin_9), J7.2 (Pin_2), U3.1 (~WAKE), U3.2 (+3.3Vaux), U3.3 (COEX1), U3.4 (GND), U3.5 (COEX2), U3.6 (+1.5V); no longer U1.10 (MICN)
- net GSM_ANT: now also C7.1, R6.2
- net MICP: now also U3.32 (SMB_DATA)
- net PWR_CNTRL: now also J2.12 (Pin_12), U3.8 (UIM_PWR)
- net PWR_KEY: now also J2.11 (Pin_11), U3.10 (UIM_DATA)
- net SIM_CLK: now also U3.44 (~LED_WLAN)
- net SIM_DATA: now also U3.46 (~LED_WPAN)
- net SIM_RST: now also U3.42 (~LED_WWAN)
- net SIM_VDD: now also D5.6, U3.48 (+1.5V)
- net SPKN: now also U3.38 (USB_D+); no longer C8.1
- net SPKP: now also U3.36 (USB_D-); no longer C7.1, C8.2
- net UART1_CTS: now also U3.23 (PERn0)
- net UART1_DCD: now also U3.21 (GND)
- net UART1_DTR: now also U3.19 (UIM_C4)
- net UART1_RI: now also U3.17 (UIM_C8)
- net UART1_RTS: now also U3.29 (GND); no longer R6.1
- net UART1_RXD: now also U3.27 (GND)
- net UART1_TXD: now also U3.25 (PERp0)
- net VDD_EXT: now also U3.12 (UIM_CLK)
- net Vin: now also SW2.2 (B), U3.11 (RefClk-), U3.13 (RefClk+), U3.15 (GND)
- net at D4.1 (K), L1.1: now also U2.2 (Out); no longer U2.4 (FB)
- net at R22.2, R25.1: now also U2.4 (FB); no longer U2.2 (Out)
- net at J1.2 (RST), R1.1: now also D5.5
- net at J1.7 (I/O), R3.1: now also D5.4
- net at R4.2: now also J2.10 (Pin_10)
- net at R5.2: now also J2.8 (Pin_8)
- net at R8.2: now also J2.7 (Pin_7)
- net at J6.SIG: now also C8.1, R6.1
- new net: J2.2 (Pin_2), J2.4 (Pin_4), SW2.1 (A)
- new net MICN: U1.10 (MICN), U3.34 (GND)
- new net Vline: J7.1 (Pin_1), SW2.3 (C)
- no-connect marks 9 -> 12
Other:
- note removed: "Audio Conn"
- moved on the sheet: J6, R11, R14, R8
